File: postal/postal.sch (KiCad schematic (older format))
At the start: 29 parts, among them J1 Conn_01x06, J2 i2c-header, U1 ATMEGA8-16AU, U2 CP2102N-A01-GQFN24, U3 AP1117-33, U4 24cXX, U5 SPI_FLASH, U6 93CxxA, Y1 14,7456

Commit message: Create pcb
Parts:
- added J3: USB_B_Micro, Connector_USB:USB_Micro-B_Molex_47346-0001, symbol Connector_Specialized:USB_B_Micro
- added R10, R9: 30, Resistor_SMD:R_0805_2012Metric, symbol postal-rescue:R-device
- added R8: 0, Resistor_SMD:R_0805_2012Metric, symbol postal-rescue:R-device
- C1, C2, C3, C4, C5, C6, C8, C9: footprint Capacitors_SMD:C_0805 -> Capacitor_SMD:C_0805_2012Metric; symbol device:C -> postal-rescue:C-device
- C10, C7: symbol device:CP -> postal-rescue:CP-device
- D1: footprint Diodes_SMD:D_MiniMELF -> Diode_SMD:D_MiniMELF; symbol device:D -> postal-rescue:D-device
- D2: footprint LEDs:LED_D3.0mm -> LED_THT:LED_D3.0mm; symbol device:LED -> postal-rescue:LED-device
- J1: footprint Pin_Headers:Pin_Header_Straight_2x03_Pitch2.54mm -> Connector_PinHeader_2.54mm:PinHeader_2x03_P2.54mm_Vertical; symbol Connector:Conn_01x06 -> postal-rescue:Conn_01x06-Connector
- J2: footprint Pin_Headers:Pin_Header_Straight_1x03_Pitch2.54mm -> Connector_PinHeader_2.54mm:PinHeader_1x03_P2.54mm_Vertical; symbol Connector:Conn_01x03 -> postal-rescue:Conn_01x03-Connector
- L1: footprint Inductors_SMD:L_0805 -> Inductor_SMD:L_0805_2012Metric; symbol device:L -> postal-rescue:L-device
- R1, R2, R3, R4, R5, R6, R7: footprint Resistors_SMD:R_0805 -> Resistor_SMD:R_0805_2012Metric; symbol device:R -> postal-rescue:R-device
- U1: footprint Housings_QFP:LQFP-32_7x7mm_Pitch0.8mm -> Package_QFP:LQFP-32_7x7mm_P0.8mm; symbol atmel:ATMEGA8-16AU -> postal-rescue:ATMEGA8-16AU-atmel
- U2: footprint Housings_DFN_QFN:QFN-24-1EP_4x4mm_Pitch0.5mm -> Package_DFN_QFN:QFN-28-1EP_5x5mm_P0.5mm; symbol silabs:CP2102N-A01-GQFN24 -> postal-rescue:CP2102N-A01-GQFN24-silabs
- U3: footprint TO_SOT_Packages_SMD:SOT-223-3_TabPin2 -> Package_TO_SOT_SMD:SOT-223-3_TabPin2; symbol regul:AP1117-33 -> postal-rescue:AP1117-33-regul
- U4: footprint Housings_DIP:DIP-8_W7.62mm -> Package_DIP:DIP-8_W7.62mm_Socket; symbol memory:AT24CS02-XHM -> postal-rescue:AT24CS02-XHM-memory
- U5: footprint Housings_DIP:DIP-8_W7.62mm -> Package_DIP:DIP-8_W7.62mm_Socket; symbol memory:25LC_EEPROM -> postal-rescue:25LC_EEPROM-memory
- U6: footprint Housings_DIP:DIP-8_W7.62mm -> Package_DIP:DIP-8_W7.62mm_Socket; symbol memory:93CxxA -> postal-rescue:93CxxA-memory
- Y1: footprint Crystals:Crystal_HC49-4H_Vertical -> Crystal:Crystal_HC49-4H_Vertical; symbol device:Crystal -> postal-rescue:Crystal-device
Connections:
- net labels added: RX, TX
- wire segments 143 -> 161
- no-connect marks 14 -> 13

Commit message: Final pcb
Parts:
- removed U2: CP2102N-A01-GQFN24, Package_DFN_QFN:QFN-28-1EP_5x5mm_P0.5mm, symbol postal-rescue:CP2102N-A01-GQFN24-silabs
- added C11, C12: 100n, Capacitor_SMD:C_0805_2012Metric, symbol postal-rescue:C-device
- added U2: CP2102, Package_DFN_QFN:QFN-28-1EP_5x5mm_P0.5mm, symbol cp2102:CP2102
- C10, C7: footprint (none) -> Capacitor_Tantalum_SMD:CP_EIA-6032-28_Kemet-C
Connections:
- wire segments 161 -> 175
- no-connect marks 13 -> 22
Changed lines of the file:
@@
 RES
-$Comp
-L postal-rescue:CP2102N-A01-GQFN24-silabs U2
-U 1 1 5A5DC772
-P 2450 3600
-F 0 "U2" H 2450 4678 50  0000 C CNN
-F 1 "CP2102N-A01-GQFN24" H 2450 4587 50  0000 C CNN
-F 2 "Package_DFN_QFN:QFN-28-1EP_5x5mm_P0.5mm" H 2900 2800 50  0001 L CNN
-F 3 "http://www.silabs.com/support%20documents/technicaldocs/cp2102n-datasheet.pdf" H 2500 2550 50  0001 C CNN
-	1    2450 3600
-	1    0    0    -1
-$EndComp
 $Comp
 L postal-rescue:Crystal-device Y1
@@
 	4700 3800 4700 3700
 $Comp
-L power:GND #PWR04
-U 1 1 5A5DE242
-P 2450 4600
-F 0 "#PWR04" H 2450 4350 50  0001 C CNN
-F 1 "GND" H 2455 4427 50  0000 C CNN
-F 2 "" H 2450 4600 50  0001 C CNN
-F 3 "" H 2450 4600 50  0001 C CNN
-	1    2450 4600
-	1    0    0    -1
-$EndComp
-Wire Wire Line
-	2450 4600 2450 4500
-$Comp
-L power:GND #PWR05
-U 1 1 5A5DE4AE
-P 2550 4600
-F 0 "#PWR05" H 2550 4350 50  0001 C CNN
-F 1 "GND" H 2555 4427 50  0000 C CNN
-F 2 "" H 2550 4600 50  0001 C CNN
-F 3 "" H 2550 4600 50  0001 C CNN
-	1    2550 4600
-	1    0    0    -1
-$EndComp
-Wire Wire Line
-	2550 4600 2550 4500
-$Comp
 L power:GND #PWR06
 U 1 1 5A5DE759
@@
 F 0 "C7" H 5618 1196 50  0000 L CNN
 F 1 "10u" H 5550 1050 50  0000 L CNN
-F 2 "" H 5538 1000 50  0001 C CNN
+F 2 "Capacitor_Tantalum_SMD:CP_EIA-6032-28_Kemet-C" H 5538 1000 50  0001 C CNN
 F 3 "" H 5500 1150 50  0001 C CNN
 	1    5500 1150
@@
 F 0 "C10" H 4668 1196 50  0000 L CNN
 F 1 "10u" H 4600 1050 50  0000 L CNN
-F 2 "" H 4588 1000 50  0001 C CNN
+F 2 "Capacitor_Tantalum_SMD:CP_EIA-6032-28_Kemet-C" H 4588 1000 50  0001 C CNN
 F 3 "" H 4550 1150 50  0001 C CNN
 	1    4550 1150
@@
 Wire Wire Line
 	8600 5700 6850 5700
-Wire Wire Line
-	3050 3300 3200 3300
-Wire Wire Line
-	3050 3400 3200 3400
-Text Label 3200 3300 0    50   ~ 0
+Text Label 3250 4000 0    50   ~ 0
 TX
-Text Label 3200 3400 0    50   ~ 0
+Text Label 3250 3900 0    50   ~ 0
 RX
 Wire Wire Line
@@
 Wire Wire Line
 	1300 4000 1500 4000
-Wire Wire Line
-	1800 4000 1850 4000
 $Comp
 L postal-rescue:R-device R10
@@
 Wire Wire Line
 	1300 4100 1500 4100
-Wire Wire Line
-	1800 4100 1850 4100
 $Comp
 L postal-rescue:R-device R8
@@
 Wire Wire Line
 	1400 3800 1300 3800
-Wire Wire Line
-	1700 3800 1800 3800
-Wire Wire Line
-	1800 3800 1800 3900
-Wire Wire Line
-	1800 3900 1850 3900
+$Comp
+L cp2102:CP2102 U2
+U 1 1 5A625495
+P 2600 3700
+F 0 "U2" H 2600 4465 50  0000 C CNN
+F 1 "CP2102" H 2600 4374 50  0000 C CNN
+F 2 "Package_DFN_QFN:QFN-28-1EP_5x5mm_P0.5mm" H 2850 4000 50  0001 C CNN
+F 3 "" H 2850 4000 50  0001 C CNN
+	1    2600 3700
+	1    0    0    -1
+$EndComp
+Wire Wire Line
+	1700 3800 1900 3800
+Wire Wire Line
+	1900 3800 1900 3700
+Wire Wire Line
+	1900 3700 2100 3700
+$Comp
+L power:GND #PWR036
+U 1 1 5A632F83
+P 2050 3450
+F 0 "#PWR036" H 2050 3200 50  0001 C CNN
+F 1 "GND" H 2055 3277 50  0001 C CNN
+F 2 "" H 2050 3450 50  0001 C CNN
+F 3 "" H 2050 3450 50  0001 C CNN
+	1    2050 3450
+	0    1    1    0
+$EndComp
+Wire Wire Line
+	2050 3450 2100 3450
+Wire Wire Line
+	1950 4000 1950 4100
+Wire Wire Line
+	1950 4100 2100 4100
+Wire Wire Line
+	1800 4000 1950 4000
+Wire Wire Line
+	1900 4100 1900 4150
+Wire Wire Line
+	1900 4150 2050 4150
+Wire Wire Line
+	2050 4150 2050 4000
+Wire Wire Line
+	2050 4000 2100 4000
+Wire Wire Line
+	1800 4100 1900 4100
+Wire Wire Line
+	3100 3900 3250 3900
+Wire Wire Line
+	3100 4000 3250 4000
+NoConn ~ 3100 3200
+NoConn ~ 3100 3300
+NoConn ~ 3100 3400
+NoConn ~ 3100 3500
+NoConn ~ 3100 3600
+NoConn ~ 3100 3700
+NoConn ~ 3100 3800
+NoConn ~ 3100 4100
+NoConn ~ 3100 4200
+Wire Wire Line
+	2100 3200 1900 3200
+Wire Wire Line
+	1900 3200 1900 3700
+Connection ~ 1900 3700
+$Comp
+L postal-rescue:C-device C11
+U 1 1 5A6B956D
+P 1600 3100
+F 0 "C11" V 1550 3300 50  0000 C CNN
+F 1 "100n" V 1650 3250 50  0000 C CNN
+F 2 "Capacitor_SMD:C_0805_2012Metric" H 1638 2950 50  0001 C CNN
+F 3 "" H 1600 3100 50  0001 C CNN
+	1    1600 3100
+	0    -1   1    0
+$EndComp
+$Comp
+L postal-rescue:C-device C12
+U 1 1 5A6C129D
+P 1600 3350
+F 0 "C12" V 1550 3550 50  0000 C CNN
+F 1 "100n" V 1650 3500 50  0000 C CNN
+F 2 "Capacitor_SMD:C_0805_2012Metric" H 1638 3200 50  0001 C CNN
+F 3 "" H 1600 3350 50  0001 C CNN
+	1    1600 3350
+	0    -1   1    0
+$EndComp
+Wire Wire Line
+	1750 3100 1900 3100
+Wire Wire Line
+	1900 3100 1900 3200
+Connection ~ 1900 3200
+Wire Wire Line
+	1750 3350 2100 3350
+$Comp
+L power:GND #PWR04
+U 1 1 5A6D154C
+P 1350 3100
+F 0 "#PWR04" H 1350 2850 50  0001 C CNN
+F 1 "GND" H 1355 2927 50  0000 C CNN
+F 2 "" H 1350 3100 50  0001 C CNN
+F 3 "" H 1350 3100 50  0001 C CNN
+	1    1350 3100
+	0    1    1    0
+$EndComp
+Wire Wire Line
+	1350 3100 1450 3100
+$Comp
+L power:GND #PWR05
+U 1 1 5A6D9981
+P 1350 3350
+F 0 "#PWR05" H 1350 3100 50  0001 C CNN
+F 1 "GND" H 1355 3177 50  0000 C CNN
+F 2 "" H 1350 3350 50  0001 C CNN
+F 3 "" H 1350 3350 50  0001 C CNN
+	1    1350 3350
+	0    1    1    0
+$EndComp
+Wire Wire Line
+	1350 3350 1450 3350
+Wire Wire Line
+	1900 900  3450 900
+Wire Wire Line
+	1900 900  1900 3100
+Connection ~ 1900 3100
 $EndSCHEMATC

Commit message: Print pcb
Parts:
- added J4: PWR, Connector_PinHeader_2.54mm:PinHeader_1x03_P2.54mm_Vertical, symbol postal-rescue:Conn_01x03-Connector
- J1: value Conn_01x06 -> SPI_FLASH
Connections:
- wire segments 175 -> 184
Other:
- moved on the sheet: C3, U3
Changed lines of the file:
@@
 P 9600 2350
 F 0 "J1" H 9680 2342 50  0000 L CNN
-F 1 "Conn_01x06" H 9680 2251 50  0000 L CNN
+F 1 "SPI_FLASH" H 9680 2251 50  0000 L CNN
 F 2 "Connector_PinHeader_2.54mm:PinHeader_2x03_P2.54mm_Vertical" H 9600 2350 50  0001 C CNN
 F 3 "~" H 9600 2350 50  0001 C CNN
@@
 L postal-rescue:AP1117-33-regul U3
 U 1 1 5A5DEDA3
-P 3900 900
-F 0 "U3" H 3900 1142 50  0000 C CNN
-F 1 "AP1117-33" H 3900 1051 50  0000 C CNN
-F 2 "Package_TO_SOT_SMD:SOT-223-3_TabPin2" H 3900 1100 50  0001 C CNN
-F 3 "http://www.diodes.com/datasheets/AP1117.pdf" H 4000 650 50  0001 C CNN
-	1    3900 900
+P 2800 900
+F 0 "U3" H 2800 1142 50  0000 C CNN
+F 1 "AP1117-33" H 2800 1051 50  0000 C CNN
+F 2 "Package_TO_SOT_SMD:SOT-223-3_TabPin2" H 2800 1100 50  0001 C CNN
+F 3 "http://www.diodes.com/datasheets/AP1117.pdf" H 2900 650 50  0001 C CNN
+	1    2800 900
 	1    0    0    -1
 $EndComp
@@
 L power:GND #PWR08
 U 1 1 5A5DEE8F
-P 3900 1350
-F 0 "#PWR08" H 3900 1100 50  0001 C CNN
-F 1 "GND" H 3905 1177 50  0000 C CNN
-F 2 "" H 3900 1350 50  0001 C CNN
-F 3 "" H 3900 1350 50  0001 C CNN
-	1    3900 1350
-	1    0    0    -1
-$EndComp
-Wire Wire Line
-	3900 1350 3900 1200
+P 2800 1350
+F 0 "#PWR08" H 2800 1100 50  0001 C CNN
+F 1 "GND" H 2805 1177 50  0000 C CNN
+F 2 "" H 2800 1350 50  0001 C CNN
+F 3 "" H 2800 1350 50  0001 C CNN
+	1    2800 1350
+	1    0    0    -1
+$EndComp
+Wire Wire Line
+	2800 1350 2800 1200
 $Comp
 L postal-rescue:C-device C3
 U 1 1 5A5DF19E
-P 3450 1150
-F 0 "C3" H 3565 1196 50  0000 L CNN
-F 1 "100n" H 3565 1105 50  0000 L CNN
-F 2 "Capacitor_SMD:C_0805_2012Metric" H 3488 1000 50  0001 C CNN
-F 3 "" H 3450 1150 50  0001 C CNN
-	1    3450 1150
+P 2350 1150
+F 0 "C3" H 2465 1196 50  0000 L CNN
+F 1 "100n" H 2465 1105 50  0000 L CNN
+F 2 "Capacitor_SMD:C_0805_2012Metric" H 2388 1000 50  0001 C CNN
+F 3 "" H 2350 1150 50  0001 C CNN
+	1    2350 1150
 	1    0    0    -1
 $EndComp
@@
 L power:GND #PWR09
 U 1 1 5A5DF732
-P 3450 1350
-F 0 "#PWR09" H 3450 1100 50  0001 C CNN
-F 1 "GND" H 3455 1177 50  0000 C CNN
-F 2 "" H 3450 1350 50  0001 C CNN
-F 3 "" H 3450 1350 50  0001 C CNN
-	1    3450 1350
-	1    0    0    -1
-$EndComp
-Wire Wire Line
-	3450 1350 3450 1300
+P 2350 1350
+F 0 "#PWR09" H 2350 1100 50  0001 C CNN
+F 1 "GND" H 2355 1177 50  0000 C CNN
+F 2 "" H 2350 1350 50  0001 C CNN
+F 3 "" H 2350 1350 50  0001 C CNN
+	1    2350 1350
+	1    0    0    -1
+$EndComp
+Wire Wire Line
+	2350 1350 2350 1300
 $Comp
 L power:GND #PWR010
@@
 	5050 1350 5050 1300
 Wire Wire Line
-	3450 1000 3450 900
-Wire Wire Line
-	3450 900  3600 900
-Wire Wire Line
-	4200 900  4550 900
+	2350 1000 2350 900
+Wire Wire Line
+	2350 900  2500 900
 Wire Wire Line
 	5050 900  5050 1000
@@
 Wire Wire Line
 	4550 1000 4550 900
-Connection ~ 4550 900
 Wire Wire Line
 	4550 900  5050 900
@@
 L power:PWR_FLAG #FLG04
 U 1 1 5A6E4BDD
-P 3450 800
-F 0 "#FLG04" H 3450 875 50  0001 C CNN
-F 1 "PWR_FLAG" H 3450 974 50  0000 C CNN
-F 2 "" H 3450 800 50  0001 C CNN
-F 3 "" H 3450 800 50  0001 C CNN
-	1    3450 800
-	1    0    0    -1
-$EndComp
-Wire Wire Line
-	3450 800  3450 900
-Connection ~ 3450 900
+P 2350 800
+F 0 "#FLG04" H 2350 875 50  0001 C CNN
+F 1 "PWR_FLAG" H 2350 974 50  0000 C CNN
+F 2 "" H 2350 800 50  0001 C CNN
+F 3 "" H 2350 800 50  0001 C CNN
+	1    2350 800
+	1    0    0    -1
+$EndComp
+Wire Wire Line
+	2350 800  2350 900
+Connection ~ 2350 900
 Wire Wire Line
 	9400 3650 9150 3650
@@
 	1350 3350 1450 3350
 Wire Wire Line
-	1900 900  3450 900
-Wire Wire Line
-	1900 900  1900 3100
+	1900 900  2350 900
+Wire Wire Line
+	1900 900  1900 1850
 Connection ~ 1900 3100
+$Comp
+L postal-rescue:Conn_01x03-Connector J4
+U 1 1 5A6F4DA8
+P 3750 1000
+F 0 "J4" H 3830 1042 50  0000 L CNN
+F 1 "PWR" H 3830 951 50  0000 L CNN
+F 2 "Connector_PinHeader_2.54mm:PinHeader_1x03_P2.54mm_Vertical" H 3750 1000 50  0001 C CNN
+F 3 "~" H 3750 1000 50  0001 C CNN
+	1    3750 1000
+	1    0    0    -1
+$EndComp
+Wire Wire Line
+	3100 900  3550 900
+Wire Wire Line
+	3550 1100 3400 1100
+Wire Wire Line
+	3400 1100 3400 1850
+Wire Wire Line
+	3400 1850 1900 1850
+Connection ~ 1900 1850
+Wire Wire Line
+	1900 1850 1900 3100
+Wire Wire Line
+	4550 900  4300 900
+Wire Wire Line
+	4300 900  4300 1300
+Wire Wire Line
+	4300 1300 3250 1300
+Wire Wire Line
+	3250 1300 3250 1000
+Wire Wire Line
+	3250 1000 3550 1000
+Connection ~ 4550 900
 $EndSCHEMATC
