File: postal/postal.kicad_pcb (KiCad board)
At the start: 2 copper layers, 27 parts, among them J1 Conn_01x06, J2 i2c-header, U1 ATMEGA8-16AU, U2 CP2102N-A01-GQFN24, U3 AP1117-33, U4 24cXX, U5 SPI_FLASH, U6 93CxxA, Y1 14,7456

Commit message: Update pcb
Parts:
- moved R7 5.72 mm to (227.3, 108.9)
- moved C9 3.81 mm to (223.5, 109.0)
- moved L1 2.30 mm to (222.6, 112.5), turned to 0 degrees
Routing:
- net Net-(C2-Pad1): track 5.69 -> 17.7 mm
- net Net-(R7-Pad2): track 19.2 -> 12.5 mm
- net Net-(C5-Pad2): track 8.08 -> 4.02 mm
- net VCC: track 132.1 -> 130.9 mm
- net GND: track 107.6 -> 106.6 mm
- net Net-(R7-Pad1): track 6.66 -> 7.66 mm
- net Net-(U1-Pad24): track 25.1 -> 24.3 mm
- net Net-(U1-Pad13): track 30.3 -> 29.6 mm
Other:
- net class Default: clearance 0.2 -> 0.15
- rule trace_clearance: 0.2 -> 0.15

Commit message: Create pcb
Parts:
- added J3: USB_B_Micro, Connector_USB:USB_Micro-B_Molex_47346-0001, B.Cu at (188.0, 123.2)
- added R10: 30, Resistor_SMD:R_0805_2012Metric, B.Cu at (197.2, 123.8)
- added R8: 0, Resistor_SMD:R_0805_2012Metric, B.Cu at (193.5, 123.8)
- added R9: 30, Resistor_SMD:R_0805_2012Metric, B.Cu at (197.2, 121.3)
- C1, C2, C3, C4, C5, C6, C8, C9: footprint Capacitors_SMD:C_0805 -> Capacitor_SMD:C_0805_2012Metric; moved to B.Cu
- D1: footprint Diodes_SMD:D_MiniMELF -> Diode_SMD:D_MiniMELF; moved to B.Cu
- D2: footprint LEDs:LED_D3.0mm -> LED_THT:LED_D3.0mm
- J1: footprint Pin_Headers:Pin_Header_Straight_2x03_Pitch2.54mm -> Connector_PinHeader_2.54mm:PinHeader_2x03_P2.54mm_Vertical
- J2: footprint Pin_Headers:Pin_Header_Straight_1x03_Pitch2.54mm -> Connector_PinHeader_2.54mm:PinHeader_1x03_P2.54mm_Vertical
- L1: footprint Inductors_SMD:L_0805 -> Inductor_SMD:L_0805_2012Metric; moved to B.Cu
- R1, R2, R3, R4, R5, R6, R7: footprint Resistors_SMD:R_0805 -> Resistor_SMD:R_0805_2012Metric; moved to B.Cu
- U1: footprint Housings_QFP:LQFP-32_7x7mm_Pitch0.8mm -> Package_QFP:LQFP-32_7x7mm_P0.8mm; moved to B.Cu
- U2: footprint Housings_DFN_QFN:QFN-24-1EP_4x4mm_Pitch0.5mm -> Package_DFN_QFN:QFN-28-1EP_5x5mm_P0.5mm; moved to B.Cu
- U3: footprint TO_SOT_Packages_SMD:SOT-223-3_TabPin2 -> Package_TO_SOT_SMD:SOT-223-3_TabPin2; moved to B.Cu
- U4, U5, U6: footprint Housings_DIP:DIP-8_W7.62mm -> Package_DIP:DIP-8_W7.62mm_Socket
- Y1: footprint Crystals:Crystal_HC49-4H_Vertical -> Crystal:Crystal_HC49-4H_Vertical
- moved J2 36.4 mm to (214.6, 129.5), turned to 180 degrees
- moved D2 35.5 mm to (203.8, 96.5), turned to 90 degrees
- moved C6 31.0 mm to (198.8, 94.9), turned to 270 degrees
- moved U3 29.2 mm to (192.4, 97.1), turned to 90 degrees
- moved U2 28.5 mm to (205.0, 123.8)
- moved C3 25.6 mm to (186.7, 98.1)
- moved R2 24.4 mm to (204.8, 103.5), turned to 0 degrees
- moved C8 20.6 mm to (233.4, 104.8), turned to 180 degrees
- moved C5 19.6 mm to (223.5, 110.8)
- moved C9 15.3 mm to (235.3, 118.7), turned to 0 degrees
- moved R7 8.52 mm to (223.5, 116.5), turned to 270 degrees
- moved C2 6.94 mm to (205.7, 114.6), turned to 90 degrees
- moved L1 6.23 mm to (223.5, 106.4), turned to 90 degrees
- moved Y1 3.61 mm to (200.7, 109.4), turned to 270 degrees
- moved R6 2.87 mm to (227.7, 92.1), turned to 0 degrees
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Connections:
- U1 pad 30: Net-(U1-Pad30) -> /RX
- U1 pad 31: Net-(U1-Pad31) -> /TX
- U2 pad 20: Net-(U2-Pad20) -> /TX
- U2 pad 21: Net-(U2-Pad21) -> /RX
Routing:
- net GND: track 106.6 -> 298.6 mm, vias 0 -> 2
- net /MISO: track 12.4 -> 99.1 mm, vias 0 -> 2
- net VCC: track 130.9 -> 171.4 mm, vias 0 -> 4
- net /SCK: track 21.6 -> 53.1 mm
- net /SCL: track 7.37 -> 38.3 mm
- net /RES: track 27.8 -> 54.7 mm, vias 0 -> 2
- net /SDA: track 5.08 -> 27.4 mm
- net Net-(U1-Pad13): track 29.6 -> 51.1 mm, vias 0 -> 2
- net Net-(R8-Pad1): track 0.00 -> 14.3 mm
- net Net-(U1-Pad24): track 24.3 -> 38.2 mm
- net /RX: track 0.00 -> 12.1 mm
- net /TX: track 0.00 -> 11.2 mm
- net Net-(R9-Pad1): track 0.00 -> 11.0 mm
- net Net-(J3-Pad3): track 0.00 -> 9.07 mm
- net Net-(J3-Pad2): track 0.00 -> 6.93 mm
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Other:
- net class Default: via_dia 0.8 -> 1.8
- net class Thin added: clearance 0.15, trace_width 0.3, via_dia 1.8, via_drill 0.4

Commit message: Final pcb
Parts:
- added C10: 10u, Capacitor_Tantalum_SMD:CP_EIA-6032-28_Kemet-C, B.Cu at (193.0, 111.1)
- added C11: 100n, Capacitor_SMD:C_0805_2012Metric, B.Cu at (193.4, 115.6)
- added C12: 100n, Capacitor_SMD:C_0805_2012Metric, B.Cu at (193.4, 118.7)
- added C7: 10u, Capacitor_Tantalum_SMD:CP_EIA-6032-28_Kemet-C, B.Cu at (221.6, 126.9)
- U2: value CP2102N-A01-GQFN24 -> CP2102
- moved C3 9.64 mm to (189.5, 107.3), turned to 180 degrees
Connections:
- C3 pad 1: Net-(C3-Pad1) -> Net-(C11-Pad2)
- R8 pad 1: Net-(R8-Pad1) -> Net-(C11-Pad2)
- U2 pad 10: Net-(U2-Pad10) -> (no net)
- U2 pad 13: Net-(U2-Pad13) -> (no net)
- U2 pad 14: Net-(U2-Pad14) -> (no net)
- U2 pad 15: Net-(U2-Pad15) -> (no net)
- U2 pad 16: Net-(U2-Pad16) -> (no net)
- U2 pad 17: Net-(U2-Pad17) -> (no net)
- U2 pad 18: Net-(U2-Pad18) -> (no net)
- U2 pad 19: Net-(U2-Pad19) -> (no net)
- U2 pad 2: GND -> Net-(U2-Pad2)
- U2 pad 20: /TX -> (no net)
- U2 pad 21: /RX -> (no net)
- U2 pad 22: Net-(U2-Pad22) -> (no net)
- U2 pad 25: GND -> /TX
- U2 pad 26: (no net) -> /RX
- U2 pad 27: (no net) -> Net-(U2-Pad27)
- U2 pad 28: (no net) -> Net-(U2-Pad28)
- U2 pad 3: Net-(R9-Pad1) -> GND
- U2 pad 4: Net-(R10-Pad1) -> Net-(R9-Pad1)
- U2 pad 5: Net-(U2-Pad5) -> Net-(R10-Pad1)
- U2 pad 7: Net-(U2-Pad7) -> Net-(C11-Pad2)
- U2 pad 8: Net-(R8-Pad1) -> Net-(C11-Pad2)
- U3 pad 3: Net-(C3-Pad1) -> Net-(C11-Pad2)
Routing:
- net Net-(C11-Pad2): track 0.00 -> 71.1 mm
- net Net-(R8-Pad1): track 14.3 -> 0.00 mm
- net Net-(C12-Pad2): track 0.00 -> 10.9 mm
- net GND: track 298.6 -> 309.0 mm
- net /RX: track 12.1 -> 20.4 mm
- net VCC: track 171.4 -> 179.6 mm
- net /TX: track 11.2 -> 18.4 mm
- net Net-(C3-Pad1): track 5.66 -> 0.00 mm
- net /SCL: track 38.3 -> 37.6 mm
Other:
- board outline added: 59 x 43 mm

Commit message: Print pcb
Parts:
- added J4: PWR, Connector_PinHeader_2.54mm:PinHeader_1x03_P2.54mm_Vertical, F.Cu at (191.0, 101.1)
- J1: value Conn_01x06 -> SPI_FLASH
- moved C6 2.29 mm to (200.0, 93.0), turned to 90 degrees
- moved U3 1.98 mm to (193.0, 95.2), turned to 180 degrees
Connections:
- U3 pad 2: VCC -> Net-(J4-Pad1)
Routing:
- net Net-(C11-Pad2): track 71.1 -> 48.6 mm
- net GND: track 309.0 -> 322.0 mm
- net Net-(J4-Pad1): track 0.00 -> 12.6 mm
Other:
- board text added: "+3,3V"
- board text added: "+5V"
- board text added: "24Cxx"
- board text added: "93Cxx"
- board text added: "BOTTOM"
- board text added: "SPI"

Commit message: Final
Parts:
- moved C6 0.33 mm to (199.7, 93.0), turned to 180 degrees
Routing:
- net VCC: track 179.2 -> 177.4 mm
- net GND: track 322.0 -> 320.4 mm
Changed lines of the file:
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@@
-(kicad_pcb (version 20171130) (host pcbnew no-vcs-found-959767c~61~ubuntu17.10.1)
+(kicad_pcb (version 20171130) (host pcbnew no-vcs-found-81642dd~61~ubuntu17.10.1)
   (general
     (thickness 1.6)
     (drawings 12)
-    (tracks 427)
+    (tracks 428)
     (zones 0)
     (modules 36)
@@
     (34 B.Paste user)
     (35 F.Paste user)
-    (36 B.SilkS user)
+    (36 B.SilkS user hide)
     (37 F.SilkS user)
     (38 B.Mask user)
@@
   )
   (module Capacitor_SMD:C_0805_2012Metric (layer B.Cu)
-    (at 200.025 93.025 90)
+    (at 199.705 92.964 180)
     (descr "Capacitor SMD 0805 (2012 Metric), square (rectangular) end terminal, IPC_7351 nominal, (Body size source: http://www.tortai-tech.com/upload/download/2011102023233369053.pdf), generated with kicad-footprint-generator")
     (tags capacitor)
     (attr smd)
-    (fp_text reference C6 (at 0 1.85 90) (layer B.SilkS)
-      (effects (font (size 1 1) (thickness 0.15)) (justify mirror))
-    )
-    (fp_text value 100n (at 0 -1.85 90) (layer B.Fab)
-      (effects (font (size 1 1) (thickness 0.15)) (justify mirror))
-    )
-    (fp_line (start -1 -0.6) (end -1 0.6) (layer B.Fab) (width 0.1))
-    (fp_line (start -1 0.6) (end 1 0.6) (layer B.Fab) (width 0.1))
-    (fp_line (start 1 0.6) (end 1 -0.6) (layer B.Fab) (width 0.1))
-    (fp_line (start 1 -0.6) (end -1 -0.6) (layer B.Fab) (width 0.1))
-    (fp_line (start -0.15 0.71) (end 0.15 0.71) (layer B.SilkS) (width 0.12))
-    (fp_line (start -0.15 -0.71) (end 0.15 -0.71) (layer B.SilkS) (width 0.12))
-    (fp_line (start -1.69 -1) (end -1.69 1) (layer B.CrtYd) (width 0.05))
-    (fp_line (start -1.69 1) (end 1.69 1) (layer B.CrtYd) (width 0.05))
-    (fp_line (start 1.69 1) (end 1.69 -1) (layer B.CrtYd) (width 0.05))
-    (fp_line (start 1.69 -1) (end -1.69 -1) (layer B.CrtYd) (width 0.05))
-    (fp_text user %R (at 0 0 90) (layer B.Fab)
-      (effects (font (size 0.5 0.5) (thickness 0.08)) (justify mirror))
-    )
-    (pad 1 smd rect (at -0.955 0 90) (size 0.97 1.5) (layers B.Cu B.Paste B.Mask)
+    (fp_text reference C6 (at 0 1.85 180) (layer B.SilkS)
+      (effects (font (size 1 1) (thickness 0.15)) (justify mirror))
+    )
+    (fp_text value 100n (at 0 -1.85 180) (layer B.Fab)
+      (effects (font (size 1 1) (thickness 0.15)) (justify mirror))
+    )
+    (fp_line (start -1 -0.6) (end -1 0.6) (layer B.Fab) (width 0.1))
+    (fp_line (start -1 0.6) (end 1 0.6) (layer B.Fab) (width 0.1))
+    (fp_line (start 1 0.6) (end 1 -0.6) (layer B.Fab) (width 0.1))
+    (fp_line (start 1 -0.6) (end -1 -0.6) (layer B.Fab) (width 0.1))
+    (fp_line (start -0.15 0.71) (end 0.15 0.71) (layer B.SilkS) (width 0.12))
+    (fp_line (start -0.15 -0.71) (end 0.15 -0.71) (layer B.SilkS) (width 0.12))
+    (fp_line (start -1.69 -1) (end -1.69 1) (layer B.CrtYd) (width 0.05))
+    (fp_line (start -1.69 1) (end 1.69 1) (layer B.CrtYd) (width 0.05))
+    (fp_line (start 1.69 1) (end 1.69 -1) (layer B.CrtYd) (width 0.05))
+    (fp_line (start 1.69 -1) (end -1.69 -1) (layer B.CrtYd) (width 0.05))
+    (fp_text user %R (at 0 0 180) (layer B.Fab)
+      (effects (font (size 0.5 0.5) (thickness 0.08)) (justify mirror))
+    )
+    (pad 1 smd rect (at -0.955 0 180) (size 0.97 1.5) (layers B.Cu B.Paste B.Mask)
       (net 28 VCC))
-    (pad 2 smd rect (at 0.955 0 90) (size 0.97 1.5) (layers B.Cu B.Paste B.Mask)
+    (pad 2 smd rect (at 0.955 0 180) (size 0.97 1.5) (layers B.Cu B.Paste B.Mask)
       (net 15 GND))
     (model ${KISYS3DMOD}/Capacitor_SMD.3dshapes/C_0805_2012Metric.wrl
@@
     )
   )
-  (gr_text +3,3V (at 190.5 104.14) (layer F.Fab)
+  (gr_text +3,3V (at 189.865 97.282) (layer F.Fab)
     (effects (font (size 1.5 1.5) (thickness 0.3)))
   )
-  (gr_text +5V (at 198.12 104.14) (layer F.Fab)
+  (gr_text +5V (at 196.85 97.155) (layer F.Fab)
     (effects (font (size 1.5 1.5) (thickness 0.3)))
   )
@@
   (via (at 211.455 104.775) (size 1.8) (drill 0.4) (layers F.Cu B.Cu) (net 8))
   (via (at 240.03 104.775) (size 1.8) (drill 0.4) (layers F.Cu B.Cu) (net 8))
+  (segment (start 196.165 92.95) (end 198.736 92.95) (width 0.4) (layer B.Cu) (net 15))
+  (segment (start 198.736 92.95) (end 198.75 92.964) (width 0.4) (layer B.Cu) (net 15))
   (segment (start 193.28 92.95) (end 192.405 92.075) (width 0.4) (layer B.Cu) (net 15))
   (segment (start 196.165 92.95) (end 193.28 92.95) (width 0.4) (layer B.Cu) (net 15))
@@
   (segment (start 187.96 92.075) (end 187.96 103.515) (width 0.4) (layer B.Cu) (net 15))
   (segment (start 187.96 103.515) (end 188.59 104.145) (width 0.4) (layer B.Cu) (net 15))
-  (segment (start 197.979 92.95) (end 198.859 92.07) (width 0.4) (layer B.Cu) (net 15))
-  (segment (start 198.859 92.07) (end 200.025 92.07) (width 0.4) (layer B.Cu) (net 15))
-  (segment (start 196.165 92.95) (end 197.979 92.95) (width 0.4) (layer B.Cu) (net 15))
   (segment (start 188.59 111.125) (end 188.59 115.645) (width 0.4) (layer B.Cu) (net 15))
   (segment (start 188.59 107.315) (end 188.59 111.125) (width 0.4) (layer B.Cu) (net 15))
@@
   (segment (start 200.66 114.3) (end 201.935 115.575) (width 0.4) (layer B.Cu) (net 21))
   (segment (start 201.935 115.575) (end 205.74 115.575) (width 0.4) (layer B.Cu) (net 21))
+  (segment (start 198.247 96.393) (end 200.914 96.393) (width 0.4) (layer B.Cu) (net 28))
+  (segment (start 200.914 96.393) (end 202.057 95.25) (width 0.4) (layer B.Cu) (net 28))
+  (segment (start 202.057 95.25) (end 202.057 93.98) (width 0.4) (layer B.Cu) (net 28))
+  (segment (start 193.929 96.393) (end 198.247 96.393) (width 0.4) (layer B.Cu) (net 28))
+  (segment (start 198.247 104.394) (end 197.612 105.029) (width 0.4) (layer B.Cu) (net 28))
+  (segment (start 198.247 96.393) (end 198.247 104.394) (width 0.4) (layer B.Cu) (net 28))
+  (segment (start 197.612 105.029) (end 197.612 111.125) (width 0.4) (layer B.Cu) (net 28))
+  (segment (start 200.66 92.964) (end 202.057 92.964) (width 0.4) (layer B.Cu) (net 28))
+  (segment (start 202.057 92.964) (end 202.057 93.98) (width 0.4) (layer B.Cu) (net 28))
   (segment (start 210.566 114.554) (end 207.391 117.729) (width 0.4) (layer B.Cu) (net 28))
   (segment (start 210.566 112.0775) (end 210.566 114.554) (width 0.4) (layer B.Cu) (net 28))
@@
   (segment (start 199.755167 117.729) (end 197.612 115.585833) (width 0.4) (layer B.Cu) (net 28))
   (segment (start 197.612 115.585833) (end 197.612 111.125) (width 0.4) (layer B.Cu) (net 28))
-  (segment (start 202.057 96.393) (end 202.057 93.98) (width 0.4) (layer B.Cu) (net 28))
   (segment (start 193.548 96.774) (end 193.929 96.393) (width 0.4) (layer B.Cu) (net 28))
-  (segment (start 202.057 100.584) (end 202.057 96.393) (width 0.4) (layer B.Cu) (net 28))
   (segment (start 193.548 101.092) (end 193.548 96.774) (width 0.4) (layer B.Cu) (net 28))
-  (segment (start 193.929 96.393) (end 202.057 96.393) (width 0.4) (layer B.Cu) (net 28))
-  (segment (start 200.025 93.98) (end 201.175 93.98) (width 0.4) (layer B.Cu) (net 28))
-  (segment (start 201.175 93.98) (end 202.057 93.98) (width 0.4) (layer B.Cu) (net 28))
-  (segment (start 197.612 105.029) (end 202.057 100.584) (width 0.4) (layer B.Cu) (net 28))
-  (segment (start 197.612 111.125) (end 197.612 105.029) (width 0.4) (layer B.Cu) (net 28))
   (segment (start 202.057 93.98) (end 203.835 93.98) (width 0.4) (layer B.Cu) (net 28))
   (segment (start 195.46 111.125) (end 196.89 111.125) (width 0.4) (layer B.Cu) (net 28))
